Commit message: Release/3.0.0

File: hsrb_description/robots/hsrb4s.urdf.xacro (robot description, xacro)
@@ -11,5 +11,4 @@
     <xacro:include filename="$(find hsrb_description)/urdf/wrist_v0/wrist.urdf.xacro" />
     <xacro:include filename="$(find hsrb_description)/urdf/hand_v0/hand.urdf.xacro" />
-    <xacro:arg name="gazebo_sim" default="False"/>
     <xacro:arg name="ignition_gazebo_sim" default="False"/>
     <xacro:arg name="rviz_sim" default="False"/>
@@ -38,11 +37,7 @@
     </xacro:hsrb_hand>
     <!-- Import ros2_control description -->
-    <xacro:if value="${not $(arg gazebo_sim) and not $(arg ignition_gazebo_sim) and not $(arg rviz_sim)}">
+    <xacro:if value="${not $(arg ignition_gazebo_sim) and not $(arg rviz_sim)}">
       <xacro:include filename="$(find hsrb_description)/urdf/ros2_control.robot.xacro" />
       <xacro:ros2_control_robot/>
-    </xacro:if>
-    <xacro:if value="$(arg gazebo_sim)">
-      <xacro:include filename="$(find hsrb_description)/urdf/ros2_control.gazebo.xacro" />
-      <xacro:ros2_contorl_gazebo/>
     </xacro:if>
     <xacro:if value="$(arg ignition_gazebo_sim)">

File: hsrb_description/urdf/common.xacro (robot description, xacro)
@@ -1,5 +1,4 @@
 <?xml version="1.0"?>
 <robot xmlns:xacro="http://ros.org/wiki/xacro">
-  <xacro:arg name="ignition_gazebo_sim" default="False" />
   <xacro:arg name="implicit_damping" default="false" />
   <xacro:macro name="gazebo_link" params="name gravity collide friction">
@@ -50,28 +49,11 @@
       <mu1>${friction}</mu1>
       <mu2>${friction}</mu2>
-      <xacro:if value="$(arg ignition_gazebo_sim)">
-        <sensor name="${name}_contact" type="contact">
-          <always_on>true</always_on>
-          <update_rate>10</update_rate>
-          <contact>
-            <collision>${name}_link_collision</collision>
-          </contact>
-        </sensor>
-      </xacro:if>
-      <xacro:unless value="$(arg ignition_gazebo_sim)">
-        <sensor name="${name}_contact" type="contact">
-          <always_on>true</always_on>
-          <update_rate>10</update_rate>
-          <contact>
-            <collision>${name}_link_collision</collision>
-          </contact>
-          <plugin name="${name}_bumper_controller" filename="libtmc_gazebo_ros_bumper.so">
-            <ros>
-              <namespace>${robot_namespace}</namespace>
-              <remapping>bumper_states:=${name}_sensor</remapping>
-            </ros>
-          </plugin>
-        </sensor>
-      </xacro:unless>
+      <sensor name="${name}_contact" type="contact">
+        <always_on>true</always_on>
+        <update_rate>10</update_rate>
+        <contact>
+          <collision>${name}_link_collision</collision>
+        </contact>
+      </sensor>
     </gazebo>
   </xacro:macro>

File: hsrb_description/urdf/ros2_control.rviz.xacro (robot description, xacro)
@@ -4,7 +4,7 @@
     <ros2_control name="GenericSystem" type="system">
       <hardware>
-        <plugin>fake_components/GenericSystem</plugin>
-        <param name="fake_sensor_commands">False</param>
-        <param name="state_following_offset">0.0</param>
+        <plugin>tmc_hardware_interface/GenericSystem</plugin>
+        <param name="mock_sensor_commands">False</param>
+        <param name="position_state_following_offset">0.0</param>
         <param name="calculate_dynamics">True</param>
       </hardware>

File: hsrb_parts_description/urdf/sensors/asus_xtion.gazebo.xacro (robot description, xacro)
@@ -12,44 +12,4 @@
     <xacro:property name="XtionFrameRate" value="30"/>
     <xacro:macro name="asus_xtion_gazebo" params="robot_namespace sensor_name parent_frame topic_frame_id">
-        <gazebo reference="${parent_frame}">
-            <sensor type="depth" name="openni_camera_camera">
-                <always_on>0</always_on>
-                <update_rate>30</update_rate>
-                <visualize>true</visualize>
-                <camera>
-                    <horizontal_fov>1.047</horizontal_fov>
-                    <image>
-                        <width>640</width>
-                        <height>480</height>
-                        <format>B8G8R8</format>
-                    </image>
-                    <depth_camera>
-                    </depth_camera>
-                    <clip>
-                        <near>0.1</near>
-                        <far>100</far>
-                    </clip>
-                </camera>
-                <plugin name="${sensor_name}_controller" filename="libgazebo_ros_camera.so">
-                    <camera_name>${sensor_name}</camera_name>
-                    <frame_name>${topic_frame_id}</frame_name>
-                    <hack_baseline>0</hack_baseline>
-                    <min_depth>0.5</min_depth>
-                    <max_depth>9.2</max_depth>
-                    <cx>0.0</cx>
-                    <cy>0.0</cy>
-                    <ros>
-                        <namespace>${robot_namespace}</namespace>
-                        <remapping>${sensor_name}/image_raw:=${sensor_name}/rgb/image_rect_color</remapping>
-                        <remapping>${sensor_name}/camera_info:=${sensor_name}/rgb/camera_info</remapping>
-                        <remapping>${sensor_name}/depth/image_raw:=${sensor_name}/depth_registered/image_rect_raw</remapping>
-                        <remapping>${sensor_name}/depth/camera_info:=${sensor_name}/depth_registered/camera_info</remapping>
-                        <remapping>${sensor_name}/points:=${sensor_name}/depth_registered/rectified_points</remapping>
-                    </ros>
-                </plugin>
-            </sensor>
-        </gazebo>
-    </xacro:macro>
-    <xacro:macro name="asus_xtion_gazebo_ignition" params="robot_namespace sensor_name parent_frame topic_frame_id">
         <gazebo reference="${parent_frame}">
             <sensor type="camera" name="openni_camera_camera_rgb">
@@ -89,4 +49,5 @@
                     </clip>
                 </camera>
+                <!-- temporal hack to fix ignition gazebo bug, see:https://github.com/gazebosim/gz-sensors/issues/29 -->
                 <gz_frame_id>${topic_frame_id}</gz_frame_id>
                 <topic>${robot_namespace}/${sensor_name}/depth_registered/image</topic>

File: hsrb_parts_description/urdf/sensors/asus_xtion.urdf.xacro (robot description, xacro)
@@ -2,5 +2,4 @@
 <robot name="hsrb" xmlns:xacro="http://ros.org/wiki/xacro">
     <xacro:include filename="$(find hsrb_parts_description)/urdf/sensors/asus_xtion.gazebo.xacro"/>
-    <xacro:arg name="ignition_gazebo_sim" default="false" />
     <!-- rgbd_sensor -->
     <xacro:macro name="asus_xtion" params="prefix parent robot_namespace sensor_name *origin">
@@ -41,18 +40,9 @@
             </inertial>
         </link>
-        <xacro:if value="$(arg ignition_gazebo_sim)">
-            <xacro:asus_xtion_gazebo_ignition
-                robot_namespace="${robot_namespace}"
-                sensor_name="${prefix}_${sensor_name}"
-                parent_frame="${prefix}_${sensor_name}_gazebo_frame"
-                topic_frame_id="${prefix}_${sensor_name}_rgb_frame" />
-        </xacro:if>
-        <xacro:unless value="$(arg ignition_gazebo_sim)">
-            <xacro:asus_xtion_gazebo
-                robot_namespace="${robot_namespace}"
-                sensor_name="${prefix}_${sensor_name}"
-                parent_frame="${prefix}_${sensor_name}_gazebo_frame"
-                topic_frame_id="${prefix}_${sensor_name}_rgb_frame" />
-        </xacro:unless>
+        <xacro:asus_xtion_gazebo
+            robot_namespace="${robot_namespace}"
+            sensor_name="${prefix}_${sensor_name}"
+            parent_frame="${prefix}_${sensor_name}_gazebo_frame"
+            topic_frame_id="${prefix}_${sensor_name}_rgb_frame" />
     </xacro:macro>
 </robot>

File: hsrb_parts_description/urdf/sensors/hokuyo_laser.gazebo.xacro (robot description, xacro)
@@ -3,66 +3,34 @@
     <xacro:arg name="gazebo_visualization_enabled" default="true" />
     <xacro:macro name="hokuyo_laser_gazebo" params="sensor_name robot_namespace ros_topic frame_name min_angle max_angle">
-        <gazebo reference="${frame_name}">
-            <sensor type="ray" name="${sensor_name}">
-                <pose>0 0 0 0 0 0</pose>
-                <update_rate>30.0</update_rate>
-                <visualize>$(arg gazebo_visualization_enabled)</visualize>
-                <ray>
-                    <scan>
-                        <horizontal>
-                            <samples>721</samples>
-                            <resolution>1</resolution>
-                            <min_angle>${min_angle}</min_angle>
-                            <max_angle>${max_angle}</max_angle>
-                        </horizontal>
-                    </scan>
-                    <range>
-                        <min>0.05</min>
-                        <max>60</max>
-                        <resolution>0.001</resolution>
-                    </range>
-                </ray>
-                <plugin name="hokuyo_laser" filename="libgazebo_ros_ray_sensor.so">
-                    <output_type>sensor_msgs/LaserScan</output_type>
-                    <frame_name>${frame_name}</frame_name>
-                    <ros>
-                        <namespace>${robot_namespace}</namespace>
-                        <remapping>~/out:=${ros_topic}</remapping>
-                    </ros>
-                </plugin>
-            </sensor>
-        </gazebo>
-    </xacro:macro>
-    <xacro:macro name="hokuyo_laser_gazebo_ignition" params="sensor_name robot_namespace ros_topic frame_name min_angle max_angle">
-        <gazebo reference="${frame_name}">
-            <sensor name="${sensor_name}" type="gpu_lidar">
-                <pose>0 0 0 0 0 0</pose>
-                <topic>${robot_namespace}/${sensor_name}/${ros_topic}</topic>
-                <gz_frame_id>${frame_name}</gz_frame_id>
-                <update_rate>30.0</update_rate>
-                <visualize>$(arg gazebo_visualization_enabled)</visualize>
-                <lidar>
-                    <scan>
-                        <horizontal>
-                            <samples>721</samples>
-                            <resolution>1</resolution>
-                            <min_angle>${min_angle}</min_angle>
-                            <max_angle>${max_angle}</max_angle>
-                        </horizontal>
-                        <vertical>
-                            <samples>1</samples>
-                            <resolution>1</resolution>
-                            <min_angle>0.0</min_angle>
-                            <max_angle>0.0</max_angle>
-                        </vertical>
-                    </scan>
-                    <range>
-                        <min>0.05</min>
-                        <max>60.0</max>
-                        <resolution>0.001</resolution>
-                    </range>
-                </lidar>
-            </sensor>
-        </gazebo>
+      <gazebo reference="${frame_name}">
+        <sensor name="${sensor_name}" type='gpu_lidar'>
+          <pose>0 0 0 0 0 0</pose>
+          <topic>${robot_namespace}/${sensor_name}/${ros_topic}</topic>
+          <gz_frame_id>${frame_name}</gz_frame_id>
+          <update_rate>30.0</update_rate>
+          <visualize>$(arg gazebo_visualization_enabled)</visualize>
+          <lidar>
+            <scan>
+              <horizontal>
+                <samples>721</samples>
+                <resolution>1</resolution>
+                <min_angle>${min_angle}</min_angle>
+                <max_angle>${max_angle}</max_angle>
+              </horizontal>
+              <vertical>
+                <samples>1</samples>
+                <resolution>1</resolution>
+                <min_angle>0.0</min_angle>
+                <max_angle>0.0</max_angle>
+              </vertical>
+            </scan>
+            <range>
+              <min>0.05</min>
+              <max>60.0</max>
+              <resolution>0.001</resolution>
+            </range>
+          </lidar>
+        </sensor>
+      </gazebo>
     </xacro:macro>
 </robot>

File: hsrb_parts_description/urdf/sensors/hokuyo_laser.urdf.xacro (robot description, xacro)
@@ -2,7 +2,6 @@
 <robot xmlns:xacro="http://ros.org/wiki/xacro">
     <xacro:include filename="$(find hsrb_parts_description)/urdf/sensors/hokuyo_laser.gazebo.xacro"/>
-    <xacro:arg name="ignition_gazebo_sim" default="false" />
     <!-- range sensor -->
-    <xacro:macro name="hokuyo_laser" params="prefix robot_namespace parent min_angle max_angle ros_topic:='scan' *origin">
+    <xacro:macro name="hokuyo_laser" params="prefix robot_namespace parent min_angle max_angle *origin">
         <joint name="${prefix}_range_sensor_joint" type="fixed">
             <xacro:insert_block name="origin" />
@@ -27,20 +26,10 @@
             </inertial>
         </link>
-        <xacro:if value="$(arg ignition_gazebo_sim)">
-            <xacro:hokuyo_laser_gazebo_ignition
-                sensor_name="${prefix}_range_sensor"
-                robot_namespace="${robot_namespace}"
-                ros_topic="${ros_topic}"
-                frame_name="${prefix}_range_sensor_link"
-                min_angle="${min_angle}" max_angle="${max_angle}" />
-        </xacro:if>
-        <xacro:unless value="$(arg ignition_gazebo_sim)">
-            <xacro:hokuyo_laser_gazebo
-                sensor_name="${prefix}_range_sensor"
-                robot_namespace="${robot_namespace}"
-                ros_topic="${ros_topic}"
-                frame_name="${prefix}_range_sensor_link"
-                min_angle="${min_angle}" max_angle="${max_angle}" />
-        </xacro:unless>
+        <xacro:hokuyo_laser_gazebo
+            sensor_name="${prefix}_range_sensor"
+            robot_namespace="${robot_namespace}"
+            ros_topic="scan"
+            frame_name="${prefix}_range_sensor_link"
+            min_angle="${min_angle}" max_angle="${max_angle}" />
     </xacro:macro>
 </robot>

File: hsrb_parts_description/urdf/sensors/imu.urdf.xacro (robot description, xacro)
@@ -1,38 +1,6 @@
 <?xml version="1.0" ?>
 <robot xmlns:xacro="http://ros.org/wiki/xacro" name="hsrb">
-    <xacro:arg name="ignition_gazebo_sim" default="false" />
     <!-- imu sensor gazebo -->
     <xacro:macro name="imu_gazebo" params="sensor_name frame_name topic_name robot_namespace">
-        <gazebo reference="${frame_name}">
-            <sensor type="imu" name="${sensor_name}">
-                <update_rate>100.0</update_rate>
-                <plugin name="${sensor_name}_plugin" filename="libgazebo_ros_imu_sensor.so">
-                    <frame_name>${personal_name}/${frame_name}</frame_name>
-                    <ros>
-                        <namespace>${robot_namespace}</namespace>
-                        <remapping>~/out:=${sensor_name}/${topic_name}</remapping>
-                    </ros>
-                </plugin>
-                <imu>
-                    <noise>
-                        <type>gaussian</type>
-                        <rate>
-                            <mean>0.0</mean>
-                            <stddev>2e-4</stddev>
-                            <bias_mean>0.0000075</bias_mean>
-                            <bias_stddev>0.0000008</bias_stddev>
-                        </rate>
-                        <accel>
-                            <mean>0.0</mean>
-                            <stddev>1.7e-2</stddev>
-                            <bias_mean>0.1</bias_mean>
-                            <bias_stddev>0.001</bias_stddev>
-                        </accel>
-                    </noise>
-                </imu>
-            </sensor>
-        </gazebo>
-    </xacro:macro>
-    <xacro:macro name="imu_gazebo_ignition" params="sensor_name frame_name topic_name robot_namespace">
         <gazebo reference="${frame_name}">
             <sensor type="imu" name="${sensor_name}">
@@ -57,18 +25,9 @@
             </inertial>
         </link>
-        <xacro:if value="$(arg ignition_gazebo_sim)">
-            <xacro:imu_gazebo_ignition
-                sensor_name="${prefix}_imu"
-                frame_name="${prefix}_imu_frame"
-                topic_name="${topic_name}"
-                robot_namespace="${robot_namespace}"/>
-        </xacro:if>
-        <xacro:unless value="$(arg ignition_gazebo_sim)">
-            <xacro:imu_gazebo
-                sensor_name="${prefix}_imu"
-                frame_name="${prefix}_imu_frame"
-                topic_name="${topic_name}"
-                robot_namespace="${robot_namespace}"/>
-        </xacro:unless>
+        <xacro:imu_gazebo
+            sensor_name="${prefix}_imu"
+            frame_name="${prefix}_imu_frame"
+            topic_name="${topic_name}"
+            robot_namespace="${robot_namespace}"/>
     </xacro:macro>
 </robot>

File: hsrb_parts_description/urdf/sensors/minebea_ft_sensor.gazebo.xacro (robot description, xacro)
@@ -2,20 +2,4 @@
 <robot name="hsrb" xmlns:xacro="http://ros.org/wiki/xacro">
     <xacro:macro name="minebea_ft_sensor_gazebo" params="robot_namespace joint_name ros_topic">
-        <gazebo reference="${joint_name}">
-            <provideFeedback>true</provideFeedback>
-        </gazebo>
-        <gazebo>
-            <plugin name="ft_sensor" filename="libgazebo_ros_ft_sensor.so">
-                <update_rate>30.0</update_rate>
-                <joint_name>${joint_name}</joint_name>
-                <robotNamespace>${robot_namespace}</robotNamespace>
-                <ros>
-                    <namespace>${robot_namespace}</namespace>
-                    <remapping>wrench:=${ros_topic}</remapping>
-                </ros>
-            </plugin>
-        </gazebo>
-    </xacro:macro>
-    <xacro:macro name="minebea_ft_sensor_gazebo_ignition" params="robot_namespace joint_name ros_topic">
         <gazebo reference="${joint_name}">
             <sensor type="force_torque" name="${joint_name}_force_torque_sensor">

File: hsrb_parts_description/urdf/sensors/minebea_ft_sensor.urdf.xacro (robot description, xacro)
@@ -2,5 +2,4 @@
 <robot name="hsrb" xmlns:xacro="http://ros.org/wiki/xacro">
     <xacro:include filename="$(find hsrb_parts_description)/urdf/sensors/minebea_ft_sensor.gazebo.xacro"/>
-    <xacro:arg name="ignition_gazebo_sim" default="false" />
     <xacro:macro name="minebea_ft_sensor" params="prefix robot_namespace parent *origin">
         <joint name="${prefix}_ft_sensor_frame_joint" type="revolute">
@@ -17,16 +16,8 @@
             </inertial>
         </link>
-        <xacro:if value="$(arg ignition_gazebo_sim)">
-            <xacro:minebea_ft_sensor_gazebo_ignition
-                robot_namespace="${robot_namespace}"
-                joint_name="${prefix}_ft_sensor_frame_joint"
-                ros_topic="${prefix}_wrench/raw"/>
-        </xacro:if>
-        <xacro:unless value="$(arg ignition_gazebo_sim)">
-            <xacro:minebea_ft_sensor_gazebo
-                robot_namespace="${robot_namespace}"
-                joint_name="${prefix}_ft_sensor_frame_joint"
-                ros_topic="${prefix}_wrench/raw"/>
-        </xacro:unless>
+        <xacro:minebea_ft_sensor_gazebo
+            robot_namespace="${robot_namespace}"
+            joint_name="${prefix}_ft_sensor_frame_joint"
+            ros_topic="${prefix}_wrench/raw" />
     </xacro:macro>
 </robot>

File: hsrb_parts_description/urdf/sensors/pointgrey_chameleon.gazebo.xacro (robot description, xacro)
@@ -2,44 +2,4 @@
 <robot name="hsrb" xmlns:xacro="http://ros.org/wiki/xacro">
     <xacro:macro name="pointgrey_chameleon_gazebo" params="sensor_name parent_frame topic_frame_id robot_namespace baseline">
-        <gazebo reference="${parent_frame}">
-            <sensor type="camera" name="${sensor_name}">
-                <update_rate>4.0</update_rate>
-                <camera name="${sensor_name}">
-                    <horizontal_fov>1.16762527</horizontal_fov>
-                    <image>
-                        <width>1280</width>
-                        <height>960</height>
-                        <format>R8G8B8</format>
-                    </image>
-                    <clip>
-                        <near>0.05</near>
-                        <far>100</far>
-                    </clip>
-                    <noise>
-                        <type>gaussian</type>
-                        <mean>0.0</mean>
-                        <stddev>0.007</stddev>
-                    </noise>
-                    <distortion>
-                        <k1>0.0</k1>
-                        <k2>0.0</k2>
-                        <k3>0.0</k3>
-                        <p1>0.0</p1>
-                        <p2>0.0</p2>
-                    </distortion>
-                </camera>
-                <plugin name="${sensor_name}_camera_controller" filename="libgazebo_ros_camera.so">
-                    <camera_name>${sensor_name}</camera_name>
-                    <frame_name>${topic_frame_id}</frame_name>
-                    <hack_baseline>${baseline}</hack_baseline>
-                    <ros>
-                        <namespace>${robot_namespace}</namespace>
-                        <remapping>${sensor_name}/image_raw:=${sensor_name}/image_rect_color</remapping>
-                    </ros>
-                </plugin>
-            </sensor>
-        </gazebo>
-    </xacro:macro>
-    <xacro:macro name="pointgrey_chameleon_gazebo_ignition" params="sensor_name parent_frame topic_frame_id robot_namespace baseline">
         <gazebo reference="${parent_frame}">
             <sensor type="camera" name="${sensor_name}">
