Commit message: Release/3.0.0

File: hsrb_parts_description/urdf/sensors/pointgrey_chameleon.urdf.xacro (robot description, xacro)
@@ -2,5 +2,4 @@
 <robot xmlns:xacro="http://ros.org/wiki/xacro">
     <xacro:include filename="$(find hsrb_parts_description)/urdf/sensors/pointgrey_chameleon.gazebo.xacro"/>
-    <xacro:arg name="ignition_gazebo_sim" default="false" />
     <xacro:macro name="pointgrey_chameleon" params="prefix parent robot_namespace *origin baseline">
         <joint name="${prefix}_camera_joint" type="fixed">
@@ -34,20 +33,10 @@
             </inertial>
         </link>
-        <xacro:if value="$(arg ignition_gazebo_sim)">
-            <xacro:pointgrey_chameleon_gazebo_ignition
-                sensor_name="${prefix}_camera"
-                parent_frame="${prefix}_camera_gazebo_frame"
-                topic_frame_id="${prefix}_camera_frame"
-                robot_namespace="${robot_namespace}"
-                baseline="${baseline}" />
-        </xacro:if>
-        <xacro:unless value="$(arg ignition_gazebo_sim)">
-            <xacro:pointgrey_chameleon_gazebo
-                sensor_name="${prefix}_camera"
-                parent_frame="${prefix}_camera_gazebo_frame"
-                topic_frame_id="${prefix}_camera_frame"
-                robot_namespace="${robot_namespace}"
-                baseline="${baseline}" />
-        </xacro:unless>
+        <xacro:pointgrey_chameleon_gazebo
+            sensor_name="${prefix}_camera"
+            parent_frame="${prefix}_camera_gazebo_frame"
+            topic_frame_id="${prefix}_camera_frame"
+            robot_namespace="${robot_namespace}"
+            baseline="${baseline}" />
     </xacro:macro>
 </robot>

File: hsrb_parts_description/urdf/sensors/wide_camera.gazebo.xacro (robot description, xacro)
@@ -1,45 +1,6 @@
 <?xml version="1.0"?>
 <robot name="hsrb" xmlns:xacro="http://ros.org/wiki/xacro">
-    <xacro:macro name="wide_camera_gazebo" params="robot_namespace sensor_name parent_frame topic_frame_id">
-        <gazebo reference="${parent_frame}">
-            <sensor type="camera" name="${sensor_name}">
-                <update_rate>10.0</update_rate>
-                <camera name="${sensor_name}">
-                    <horizontal_fov>2.00</horizontal_fov>
-                    <image>
-                        <width>640</width>
-                        <height>480</height>
-                        <format>R8G8B8</format>
-                    </image>
-                    <clip>
-                        <near>0.01</near>
-                        <far>100</far>
-                    </clip>
-                    <noise>
-                        <type>gaussian</type>
-                        <mean>0.0</mean>
-                        <stddev>0.007</stddev>
-                    </noise>
-                    <distortion>
-                        <k1>0.0</k1>
-                        <k2>0.0</k2>
-                        <k3>0.0</k3>
-                        <p1>0.0</p1>
-                        <p2>0.0</p2>
-                    </distortion>
-                </camera>
-                <plugin name="${sensor_name}_camera_controller"
-                    filename="libgazebo_ros_camera.so">
-                    <camera_name>${sensor_name}</camera_name>
-                    <frame_name>${topic_frame_id}</frame_name>
-                    <hack_baseline>0.07</hack_baseline>
-                    <ros>
-                        <namespace>${robot_namespace}</namespace>
-                    </ros>
-                </plugin>
-            </sensor>
-        </gazebo>
-    </xacro:macro>
-    <xacro:macro name="wide_camera_gazebo_ignition" params="robot_namespace sensor_name parent_frame topic_frame_id">
+    <xacro:macro name="wide_camera_gazebo"
+        params="robot_namespace sensor_name parent_frame topic_frame_id">
         <gazebo reference="${parent_frame}">
             <sensor type="camera" name="${sensor_name}">

File: hsrb_parts_description/urdf/sensors/wide_camera.urdf.xacro (robot description, xacro)
@@ -2,5 +2,4 @@
 <robot xmlns:xacro="http://ros.org/wiki/xacro">
     <xacro:include filename="$(find hsrb_parts_description)/urdf/sensors/wide_camera.gazebo.xacro"/>
-    <xacro:arg name="ignition_gazebo_sim" default="false" />
     <!-- wide rgb camera -->
     <xacro:macro name="wide_camera" params="prefix parent robot_namespace rpy *origin">
@@ -29,18 +28,10 @@
             </inertial>
         </link>
-        <xacro:if value="$(arg ignition_gazebo_sim)">
-            <xacro:wide_camera_gazebo_ignition
-                robot_namespace="${robot_namespace}"
-                sensor_name="${prefix}_camera"
-                parent_frame="${prefix}_camera_gazebo_frame"
-                topic_frame_id="${prefix}_camera_frame" />
-        </xacro:if>
-        <xacro:unless value="$(arg ignition_gazebo_sim)">
-            <xacro:wide_camera_gazebo
-                robot_namespace="${robot_namespace}"
-                sensor_name="${prefix}_camera"
-                parent_frame="${prefix}_camera_gazebo_frame"
-                topic_frame_id="${prefix}_camera_frame" />
-        </xacro:unless>
+        <xacro:wide_camera_gazebo
+            robot_namespace="${robot_namespace}"
+            sensor_name="${prefix}_camera"
+            parent_frame="${prefix}_camera_gazebo_frame"
+            topic_frame_id="${prefix}_camera_frame"
+            />
     </xacro:macro>
 </robot>

File: hsrc_description/robots/hsrc1s.urdf.xacro (robot description, xacro)
@@ -15,5 +15,4 @@
     <xacro:include filename="$(find hsrc_description)/urdf/wrist_v0/wrist.urdf.xacro" />
     <xacro:include filename="$(find hsrc_description)/urdf/hand_v0/hand.urdf.xacro" />
-    <xacro:arg name="gazebo_sim" default="False"/>
     <xacro:arg name="ignition_gazebo_sim" default="False"/>
     <xacro:arg name="rviz_sim" default="False"/>
@@ -42,11 +41,7 @@
     </xacro:hsrb_hand>
     <!-- Import ros2_control description -->
-    <xacro:if value="${not $(arg gazebo_sim) and not $(arg ignition_gazebo_sim) and not $(arg rviz_sim)}">
+    <xacro:if value="${not $(arg ignition_gazebo_sim) and not $(arg rviz_sim)}">
       <xacro:include filename="$(find hsrc_description)/urdf/ros2_control.robot.xacro" />
       <xacro:ros2_control_robot/>
-    </xacro:if>
-    <xacro:if value="$(arg gazebo_sim)">
-      <xacro:include filename="$(find hsrc_description)/urdf/ros2_control.gazebo.xacro" />
-      <xacro:ros2_contorl_gazebo/>
     </xacro:if>
     <xacro:if value="$(arg ignition_gazebo_sim)">

File: hsrc_description/urdf/common.xacro (robot description, xacro)
@@ -1,5 +1,4 @@
 <?xml version="1.0"?>
 <robot xmlns:xacro="http://ros.org/wiki/xacro">
-  <xacro:arg name="ignition_gazebo_sim" default="False" />
   <xacro:arg name="implicit_damping" default="false" />
   <xacro:macro name="hsrb_position_joint_transmission" params="joint reduction">
@@ -86,28 +85,11 @@
       <mu1>${friction}</mu1>
       <mu2>${friction}</mu2>
-      <xacro:if value="$(arg ignition_gazebo_sim)">
-        <sensor name="${name}_contact" type="contact">
-          <always_on>true</always_on>
-          <update_rate>10</update_rate>
-          <contact>
-            <collision>${name}_link_collision</collision>
-          </contact>
-        </sensor>
-      </xacro:if>
-      <xacro:unless value="$(arg ignition_gazebo_sim)">
-        <sensor name="${name}_contact" type="contact">
-          <always_on>true</always_on>
-          <update_rate>10</update_rate>
-          <contact>
-            <collision>${name}_link_collision</collision>
-          </contact>
-          <plugin name="${name}_bumper_controller" filename="libtmc_gazebo_ros_bumper.so">
-            <ros>
-              <namespace>${robot_namespace}</namespace>
-              <remapping>bumper_states:=${name}_sensor</remapping>
-            </ros>
-          </plugin>
-        </sensor>
-      </xacro:unless>
+      <sensor name="${name}_contact" type="contact">
+        <always_on>true</always_on>
+        <update_rate>10</update_rate>
+        <contact>
+          <collision>${name}_link_collision</collision>
+        </contact>
+      </sensor>
     </gazebo>
   </xacro:macro>
